File: MainBoard.sch (KiCad schematic (older format))
At the start: 12 parts

Commit message: main board update
Parts:
- added C10, C11: 1uF, Capacitors_SMD:C_0805, symbol C
- added C12: C, Capacitors_SMD:C_0603, symbol C
- added C3: 3.9nF, Capacitors_SMD:C_0603, symbol C
- added C4: 10nF, Capacitors_SMD:C_0603, symbol C
- added C5: 22uF/10V, Capacitors_SMD:C_0805, symbol C
- added D1, D2: LED, LEDs:LED_0805, symbol LED
- added J1: DB25, Connect:DB25FC, symbol DB25
- added L1: 10uH/4A, footprint:ASPI-0630LR, symbol L_Small
- added Q1, Q2: BSS138, TO_SOT_Packages_SMD:SOT-23, symbol BSS138
- added R10, R11, R12, R5, R8, R9: 10k, Capacitors_SMD:C_0603, symbol R
- added R2: 6.8k, Capacitors_SMD:C_0603, symbol R
- added R3: 10k 1%, Capacitors_SMD:C_0603, symbol R
- added R4: 44.2k 1%, Capacitors_SMD:C_0603, symbol R
- added R6, R7: 330, Capacitors_SMD:C_0603, symbol R
- added RN1, RN2, RN3: 20k, Resistors_SMD:R_Array_Concave_4x0603, symbol R_Pack04
- added U6: TLV1117LV33, TO_SOT_Packages_SMD:SOT-223, symbol TLV1117LV33
- added U7: TENDA_P200, footprint:Tenda_p200, symbol TENDA_P200
- added U8: pca9685, Housings_SSOP:TSSOP-28_4.4x9.7mm_Pitch0.65mm, symbol pca9685
- C1: renamed from C?; value CP1 -> 10uF/25V; footprint (none) -> Capacitors_SMD:C_1206; Part # (none) -> 445-8867-1-ND; Vender (none) -> DigiKey
- C2: renamed from C?; value C -> 0.1uF; footprint (none) -> Capacitors_SMD:C_0603
- R1: renamed from R?; value R -> 100k; footprint (none) -> Capacitors_SMD:C_0603
- U1: renamed from U?; footprint (none) -> Housings_SOIC:SOIC-8-1EP_3.9x4.9mm_Pitch1.27mm; Part # (none) -> 946-MP2307DNLF; Vender (none) -> Mouser
- gave numbers to parts that had none: 8
Connections:
- net labels added: 3V3, 5V, SCL_3V3, SCL_5V, SDA_3V3, SDA_5V, T+
- wire segments 31 -> 109
- no-connect marks 0 -> 6
Other:
- note added: "3.3V Regulator"
- note added: "3.3V to 5V level shifter"
- note added: "5V Regulator"
- note added: "BLDC ESC X 4"
- note added: "Homplug"
- note added: "PWM Generator"
- moved on the sheet: C1, C2, C6, C7, C8, C9, R1, U1, U2, U3, U4, U5

Commit message: First layout finish
Parts:
- added C13, C14: 33uF, Capacitors_SMD:C_0603, symbol C
- added C15, C16, C17, C18: 1uF, Capacitors_SMD:C_0603, symbol C
- added D? (x2): LED, LEDs:LED_0805, symbol LED
- added P1: BOOT, Socket_Strips:Socket_Strip_Straight_1x02, symbol CONN_01X02
- added P10, P11, P12, P13, P9: CONN_01X03, Socket_Strips:Socket_Strip_Straight_1x03, symbol CONN_01X03
- added P14, P8: CONN_01X02, Socket_Strips:Socket_Strip_Straight_1x02, symbol CONN_01X02
- added P15: CONN_02X08, Socket_Strips:Socket_Strip_Straight_2x08, symbol CONN_02X08
- added P16: CONN_02X05, Socket_Strips:Socket_Strip_Straight_2x05, symbol CONN_02X05
- added P2: CONN_01X04, Connectors_JST:JST_XH_B04B-XH-A_04x2.50mm_Straight, symbol CONN_01X04
- added P3: CONN_01X05, Connectors_JST:JST_XH_B05B-XH-A_05x2.50mm_Straight, symbol CONN_01X05
- added P4, P5, P6, P7: HOLE, Connect:1pin, symbol CONN_01X01_MALE
- added Q3: DMN65D8L, TO_SOT_Packages_SMD:SOT-23, symbol Q_NMOS_GSD
- added R13, R14, R15, R16: 10k, Capacitors_SMD:C_0603, symbol R
- added R17: 1k, Capacitors_SMD:C_0603, symbol R
- added R? (x2): 330, Capacitors_SMD:C_0603, symbol R
- added RN4: 20k, Resistors_SMD:R_Array_Concave_4x0603, symbol R_Pack04
- added SW1: RESET, footprint:smd_push, symbol SW_PUSH_SMALL_H
- added U10: SI4425DDY, SMD_Packages:SOIC-8-N, symbol SI4425DDY
- added U9: STM32F103CBT6, Housings_QFP:LQFP-48_7x7mm_Pitch0.5mm, symbol STM32F103CBTx
- added Y1: 8MHz, footprint:crystal_maple, symbol Crystal_GND3_Small
Connections:
- net labels added: ESC1, ESC2, ESC3, ESC4, LED1, LED2, OSC_IN, OSC_OUT, PWR_SW, RX1, TX1
- net labels removed: CH1, CH2, CH3, CH4
- wire segments 109 -> 206
- no-connect marks 6 -> 9
Other:
- note added: "External\nPower"
- note added: "Power Control"
- note added: "Power\nSwitch"
- moved on the sheet: J1

Commit message: First layout finish
Parts:
- gave numbers to parts that had none: 4
Changed lines of the file:
@@
 $EndComp
 $Comp
-L GND #PWR8
+L GND #PWR01
 U 1 1 586CA451
 P 4075 850
-F 0 "#PWR8" H 4075 600 50  0001 C CNN
+F 0 "#PWR01" H 4075 600 50  0001 C CNN
 F 1 "GND" H 4075 700 50  0000 C CNN
 F 2 "" H 4075 850 50  0000 C CNN
@@
 $EndComp
 $Comp
-L GND #PWR9
+L GND #PWR02
 U 1 1 586CA58E
 P 4075 1625
-F 0 "#PWR9" H 4075 1375 50  0001 C CNN
+F 0 "#PWR02" H 4075 1375 50  0001 C CNN
 F 1 "GND" H 4075 1475 50  0000 C CNN
 F 2 "" H 4075 1625 50  0000 C CNN
@@
 $EndComp
 $Comp
-L GND #PWR10
+L GND #PWR03
 U 1 1 586CA67F
 P 4075 2400
-F 0 "#PWR10" H 4075 2150 50  0001 C CNN
+F 0 "#PWR03" H 4075 2150 50  0001 C CNN
 F 1 "GND" H 4075 2250 50  0000 C CNN
 F 2 "" H 4075 2400 50  0000 C CNN
@@
 $EndComp
 $Comp
-L GND #PWR11
+L GND #PWR04
 U 1 1 586CA79E
 P 4075 3200
-F 0 "#PWR11" H 4075 2950 50  0001 C CNN
+F 0 "#PWR04" H 4075 2950 50  0001 C CNN
 F 1 "GND" H 4075 3050 50  0000 C CNN
 F 2 "" H 4075 3200 50  0000 C CNN
@@
 $EndComp
 $Comp
-L GND #PWR4
+L GND #PWR05
 U 1 1 586DE565
 P 1025 2600
-F 0 "#PWR4" H 1025 2350 50  0001 C CNN
+F 0 "#PWR05" H 1025 2350 50  0001 C CNN
 F 1 "GND" H 1030 2427 50  0000 C CNN
 F 2 "" H 1025 2600 50  0000 C CNN
@@
 $EndComp
 $Comp
-L GND #PWR6
+L GND #PWR06
 U 1 1 586F0E2B
 P 2100 3825
-F 0 "#PWR6" H 2100 3575 50  0001 C CNN
+F 0 "#PWR06" H 2100 3575 50  0001 C CNN
 F 1 "GND" H 2105 3652 50  0000 C CNN
 F 2 "" H 2100 3825 50  0000 C CNN
@@
 3V3
 $Comp
-L GND #PWR5
+L GND #PWR07
 U 1 1 586F2B71
 P 1125 4850
-F 0 "#PWR5" H 1125 4600 50  0001 C CNN
+F 0 "#PWR07" H 1125 4600 50  0001 C CNN
 F 1 "GND" V 1130 4722 50  0000 R CNN
 F 2 "" H 1125 4850 50  0000 C CNN
@@
 $EndComp
 $Comp
-L GND #PWR1
+L GND #PWR08
 U 1 1 586F3827
 P 700 5250
-F 0 "#PWR1" H 700 5000 50  0001 C CNN
+F 0 "#PWR08" H 700 5000 50  0001 C CNN
 F 1 "GND" V 600 5275 50  0000 R CNN
 F 2 "" H 700 5250 50  0000 C CNN
@@
 $EndComp
 $Comp
-L GND #PWR13
+L GND #PWR09
 U 1 1 586E52C1
 P 7175 2425
-F 0 "#PWR13" H 7175 2175 50  0001 C CNN
+F 0 "#PWR09" H 7175 2175 50  0001 C CNN
 F 1 "GND" V 7100 2575 50  0000 R CNN
 F 2 "" H 7175 2425 50  0000 C CNN
@@
 3.3V to 5V level shifter
 $Comp
-L GND #PWR7
+L GND #PWR010
 U 1 1 586F313A
 P 3600 4850
-F 0 "#PWR7" H 3600 4600 50  0001 C CNN
+F 0 "#PWR010" H 3600 4600 50  0001 C CNN
 F 1 "GND" V 3475 4875 50  0000 R CNN
 F 2 "" H 3600 4850 50  0000 C CNN
@@
 $EndComp
 $Comp
-L GND #PWR18
+L GND #PWR011
 U 1 1 5870CE06
 P 11250 5675
-F 0 "#PWR18" H 11250 5425 50  0001 C CNN
+F 0 "#PWR011" H 11250 5425 50  0001 C CNN
 F 1 "GND" V 11255 5547 50  0000 R CNN
 F 2 "" H 11250 5675 50  0000 C CNN
@@
 OSC_OUT
 $Comp
-L GND #PWR16
+L GND #PWR012
 U 1 1 5870F340
 P 9200 7575
-F 0 "#PWR16" H 9200 7325 50  0001 C CNN
+F 0 "#PWR012" H 9200 7325 50  0001 C CNN
 F 1 "GND" V 9205 7447 50  0000 R CNN
 F 2 "" H 9200 7575 50  0000 C CNN
@@
 $EndComp
 $Comp
-L GND #PWR19
+L GND #PWR013
 U 1 1 587100CE
 P 12450 9400
-F 0 "#PWR19" H 12450 9150 50  0001 C CNN
+F 0 "#PWR013" H 12450 9150 50  0001 C CNN
 F 1 "GND" H 12455 9227 50  0000 C CNN
 F 2 "" H 12450 9400 50  0000 C CNN
@@
 $EndComp
 $Comp
-L GND #PWR15
+L GND #PWR014
 U 1 1 58707C58
 P 8500 6075
-F 0 "#PWR15" H 8500 5825 50  0001 C CNN
+F 0 "#PWR014" H 8500 5825 50  0001 C CNN
 F 1 "GND" V 8505 5947 50  0000 R CNN
 F 2 "" H 8500 6075 50  0000 C CNN
@@
 $EndComp
 $Comp
-L GND #PWR14
+L GND #PWR015
 U 1 1 5870F77D
 P 7575 6725
-F 0 "#PWR14" H 7575 6475 50  0001 C CNN
+F 0 "#PWR015" H 7575 6475 50  0001 C CNN
 F 1 "GND" V 7580 6597 50  0000 R CNN
 F 2 "" H 7575 6725 50  0000 C CNN
@@
 5V
 $Comp
-L GND #PWR2
+L GND #PWR016
 U 1 1 58714412
 P 850 7825
-F 0 "#PWR2" H 850 7575 50  0001 C CNN
+F 0 "#PWR016" H 850 7575 50  0001 C CNN
 F 1 "GND" V 855 7697 50  0000 R CNN
 F 2 "" H 850 7825 50  0000 C CNN
@@
 $EndComp
 $Comp
-L GND #PWR3
+L GND #PWR017
 U 1 1 5872A00C
 P 850 8100
-F 0 "#PWR3" H 850 7850 50  0001 C CNN
+F 0 "#PWR017" H 850 7850 50  0001 C CNN
 F 1 "GND" V 855 7972 50  0000 R CNN
 F 2 "" H 850 8100 50  0000 C CNN
@@
 $EndComp
 $Comp
-L GND #PWR17
+L GND #PWR018
 U 1 1 587557A0
 P 10400 2600
-F 0 "#PWR17" H 10400 2350 50  0001 C CNN
+F 0 "#PWR018" H 10400 2350 50  0001 C CNN
 F 1 "GND" H 10405 2427 50  0000 C CNN
 F 2 "" H 10400 2600 50  0000 C CNN
@@
 Connection ~ 4200 4900
 $Comp
-L GND #PWR12
+L GND #PWR019
 U 1 1 58769C9F
 P 4200 5300
-F 0 "#PWR12" H 4200 5050 50  0001 C CNN
+F 0 "#PWR019" H 4200 5050 50  0001 C CNN
 F 1 "GND" H 4205 5127 50  0000 C CNN
 F 2 "" H 4200 5300 50  0000 C CNN
@@
 $EndComp
 $Comp
-L LED D?
+L LED D3
 U 1 1 5877F101
 P 15600 8500
-F 0 "D?" H 15600 8600 50  0000 C CNN
+F 0 "D3" H 15600 8600 50  0000 C CNN
 F 1 "LED" H 15725 8450 50  0000 C CNN
 F 2 "LEDs:LED_0805" H 15591 8625 50  0001 C CNN
@@
 $EndComp
 $Comp
-L R R?
+L R R18
 U 1 1 5877F107
 P 15600 8900
-F 0 "R?" V 15525 8900 50  0000 C CNN
+F 0 "R18" V 15525 8900 50  0000 C CNN
 F 1 "330" V 15600 8900 50  0000 C CNN
 F 2 "Capacitors_SMD:C_0603" V 15530 8900 50  0001 C CNN
@@
 	15600 8650 15600 8750
 $Comp
-L GND #PWR?
+L GND #PWR020
 U 1 1 58782956
 P 15600 9050
-F 0 "#PWR?" H 15600 8800 50  0001 C CNN
+F 0 "#PWR020" H 15600 8800 50  0001 C CNN
 F 1 "GND" H 15605 8877 50  0000 C CNN
 F 2 "" H 15600 9050 50  0000 C CNN
@@
 $EndComp
 $Comp
-L LED D?
+L LED D4
 U 1 1 58783046
 P 15800 8500
-F 0 "D?" H 15800 8600 50  0000 C CNN
+F 0 "D4" H 15800 8600 50  0000 C CNN
 F 1 "LED" H 15925 8450 50  0000 C CNN
 F 2 "LEDs:LED_0805" H 15791 8625 50  0001 C CNN
@@
 Connection ~ 15800 8275
 $Comp
-L R R?
+L R R19
 U 1 1 587832D5
 P 15800 8900
-F 0 "R?" V 15725 8900 50  0000 C CNN
+F 0 "R19" V 15725 8900 50  0000 C CNN
 F 1 "330" V 15800 8900 50  0000 C CNN
 F 2 "Capacitors_SMD:C_0603" V 15730 8900 50  0001 C CNN
@@
 	15800 8650 15800 8750
 $Comp
-L GND #PWR?
+L GND #PWR021
 U 1 1 5878356B
 P 15800 9050
-F 0 "#PWR?" H 15800 8800 50  0001 C CNN
+F 0 "#PWR021" H 15800 8800 50  0001 C CNN
 F 1 "GND" H 15805 8877 50  0000 C CNN
 F 2 "" H 15800 9050 50  0000 C CNN

Commit message: First layout finish
Parts:
- removed RN4: 20k, Resistors_SMD:R_Array_Concave_4x0603, symbol R_Pack04
- added P17: CONN_01X04, Connectors_JST:JST_XH_B04B-XH-A_04x2.50mm_Straight, symbol CONN_01X04
- added P18: CONN_01X03, Socket_Strips:Socket_Strip_Straight_1x03, symbol CONN_01X03
- P15: value CONN_02X08 -> CONN_02X07; footprint Socket_Strips:Socket_Strip_Straight_2x08 -> Socket_Strips:Socket_Strip_Straight_2x07; symbol CONN_02X08 -> CONN_02X07
Connections:
- net labels added: CH1, CH2, CH3, CH4, CH5, CH6, PA0, PA1, PA11, PA12, PA13, PA14, PA15, PA2, PA3, PA4, PA5, PA6, PA7, PA8, PB12, PB13, PB14, PB15, PB3, PB4, PB5, PB6, PB7, PB8, PB9
- wire segments 206 -> 295
- no-connect marks 9 -> 14
Other:
- note added: "Connection Pins"
- moved on the sheet: C13, C14, C15, C16, C17, C18, D3, D4, J1, P1, P16, P4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
